File: console-cape.sch (KiCad schematic (older format))
At the start: 19 parts, among them J1 LCD HEADER, J2 FTDI, J3 ISP-2560, J4 DIGOUT1, J5 DIGOUT2, J6 LCD TEST, J7 CONN_01X02, U2 ATMEGA328, X1 16MHz 18pF

Commit message: added header to get GND and 3V3 from BBB P9
Parts:
- added J8: CONN_02X02, Wickerlib:CONN-HEADER-STRAIGHT-P2.54MM-2x02, symbol CONN_02X02
Connections:
- net +5V: now also J8.3 (P3), J8.4 (P4)
- net GND: now also J8.1 (P1), J8.2 (P2)
Changed lines of the file:
@@
 LIBS:valves
 LIBS:wickerlib
+LIBS:console-cape-cache
 EELAYER 25 0
 EELAYER END
@@
 Text Label 9715 1435 0    60   ~ 0
 MISO
+$Comp
+L CONN_02X02 J8
+U 1 1 59B24DD3
+P 2550 1020
+F 0 "J8" H 2550 1170 50  0000 C CNN
+F 1 "CONN_02X02" H 2550 870 50  0000 C CNN
+F 2 "Wickerlib:CONN-HEADER-STRAIGHT-P2.54MM-2x02" H 2550 -180 50  0001 C CNN
+F 3 "" H 2550 -180 50  0001 C CNN
+	1    2550 1020
+	0    -1   -1   0
+$EndComp
+$Comp
+L +5V #PWR020
+U 1 1 59B25235
+P 2600 770
+F 0 "#PWR020" H 2600 620 50  0001 C CNN
+F 1 "+5V" H 2600 910 50  0000 C CNN
+F 2 "" H 2600 770 50  0000 C CNN
+F 3 "" H 2600 770 50  0000 C CNN
+	1    2600 770
+	1    0    0    -1
+$EndComp
+$Comp
+L +5V #PWR021
+U 1 1 59B252DA
+P 2600 1270
+F 0 "#PWR021" H 2600 1120 50  0001 C CNN
+F 1 "+5V" H 2600 1410 50  0000 C CNN
+F 2 "" H 2600 1270 50  0000 C CNN
+F 3 "" H 2600 1270 50  0000 C CNN
+	1    2600 1270
+	-1   0    0    1
+$EndComp
+$Comp
+L GND #PWR022
+U 1 1 59B2555B
+P 2500 770
+F 0 "#PWR022" H 2500 520 50  0001 C CNN
+F 1 "GND" H 2500 620 50  0000 C CNN
+F 2 "" H 2500 770 50  0000 C CNN
+F 3 "" H 2500 770 50  0000 C CNN
+	1    2500 770
+	-1   0    0    1
+$EndComp
+$Comp
+L GND #PWR023
+U 1 1 59B25656
+P 2500 1270
+F 0 "#PWR023" H 2500 1020 50  0001 C CNN
+F 1 "GND" H 2500 1120 50  0000 C CNN
+F 2 "" H 2500 1270 50  0000 C CNN
+F 3 "" H 2500 1270 50  0000 C CNN
+	1    2500 1270
+	1    0    0    -1
+$EndComp
 $EndSCHEMATC
